Commit message: 加入了urdf模型缩放程序，将Heron M300的尺寸做的更加拟真

File: src/usv_world_model/urdf/heron.urdf (robot description, URDF)
Before this commit: robot WAM-V, 6 links, 5 joints
Links:
- link wamv/dummy_link: geometry collision box size=0.65 0.2 0.1; collision box size=0.65 0.2 0.1
- link wamv/left_engine_link: geometry collision box size=0.12 0.15 0.12; collision box size=0.2 0.15 0.83
- link wamv/left_propeller_link: geometry collision cylinder length=0.18 radius=0.24; visual mesh filename=package://wamv_description/models/propeller/mesh/propeller.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 scale=0.265306 0.408333 0.408333
- link wamv/right_engine_link: geometry collision box size=0.12 0.15 0.12; collision box size=0.2 0.15 0.83
- link wamv/right_propeller_link: geometry collision cylinder length=0.18 radius=0.24; visual mesh filename=package://wamv_description/models/propeller/mesh/propeller.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 scale=0.265306 0.408333 0.408333
Joints:
- joint wamv/left_chasis_engine_joint: origin xyz=-0.65 0.37 0.318237 rpy=0.0 0.0 0.0 -> xyz=-0.6 0.37 0.11 rpy=0.0 0.0 0.0
- joint wamv/left_engine_propeller_joint: origin xyz=-0.278156 0 -0.509371 rpy=0 0 0 -> xyz=-0.019579 0.000000 -0.084930 rpy=0 0 0
- joint wamv/right_chasis_engine_joint: origin xyz=-0.65 -0.37 0.318237 rpy=0.0 0.0 0.0 -> xyz=-0.6 -0.37 0.11 rpy=0.0 0.0 0.0
- joint wamv/right_engine_propeller_joint: origin xyz=-0.278156 0 -0.509371 rpy=0 0 0 -> xyz=-0.019579 0.000000 -0.084930 rpy=0 0 0

Commit message: 基本实现了MPPI MPC控制的闭环逻辑

File: src/usv_world_model/urdf/heron.urdf (robot description, URDF)
Before this commit: robot WAM-V, 6 links, 5 joints
Links:
- link wamv/left_engine_link: mass 0.1 -> 0.01
- link wamv/left_propeller_link: mass 0.1 -> 0.01
- link wamv/right_engine_link: mass 0.1 -> 0.01
- link wamv/right_propeller_link: mass 0.1 -> 0.01
